File: rs485.kicad_sch (KiCad schematic)
At the start: 7 parts, among them J1 Screw_Terminal_01x04, U27 SP3485EN-L/TR

Commit message: Implemented fixes/changes after @manawyrm review
Parts:
- removed JP2: DMX+Termination, Jumper:SolderJumper-2_P1.3mm_Open_RoundedPad1.0x1.5mm, symbol Jumper:Jumper_2_Open
- removed R114: 120, Resistor_SMD:R_0402_1005Metric, symbol Device:R
Connections:
- net DMX+: now also R113.2
- net GND: no longer R113.2
Changed lines of the file:
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@@
   (junction (at 104.775 45.72) (diameter 0) (color 0 0 0 0)
   )
-  (junction (at 82.55 41.91) (diameter 0) (color 0 0 0 0)
-  )
   (wire (pts (xy 51.435 41.91) (xy 53.975 41.91))
     (stroke (width 0) (type default))
   )
-  (wire (pts (xy 71.755 41.91) (xy 82.55 41.91))
+  (wire (pts (xy 71.755 41.91) (xy 84.455 41.91))
     (stroke (width 0) (type default))
   )
@@
     (stroke (width 0) (type default))
   )
-  (wire (pts (xy 82.55 41.91) (xy 84.455 41.91))
-    (stroke (width 0) (type default))
-  )
   (wire (pts (xy 51.435 46.99) (xy 53.975 46.99))
     (stroke (width 0) (type default))
@@
     (stroke (width 0) (type default))
   )
-  (wire (pts (xy 82.55 36.83) (xy 82.55 41.91))
-    (stroke (width 0) (type default))
-  )
   (wire (pts (xy 104.775 45.72) (xy 104.775 48.26))
     (stroke (width 0) (type default))
@@
   )
   (label "DMX-" (at 102.87 43.18 180) (fields_autoplaced)
+    (effects (font (size 1.27 1.27)) (justify right bottom))
+  )
+  (label "DMX+" (at 82.55 65.405 270) (fields_autoplaced)
     (effects (font (size 1.27 1.27)) (justify right bottom))
   )
@@
     )
   )
-  (symbol (lib_id "power:GND") (at 82.55 19.05 180) (unit 1)
-    (in_bom yes) (on_board yes) (dnp no) (fields_autoplaced)
-    (property "Reference" "#PWR057" (at 82.55 12.7 0)
-      (effects (font (size 1.27 1.27)) hide)
-    )
-    (property "Value" "GND" (at 82.55 15.24 0)
-      (effects (font (size 1.27 1.27)))
-    )
-    (property "Footprint" "" (at 82.55 19.05 0)
-      (effects (font (size 1.27 1.27)) hide)
-    )
-    (property "Datasheet" "" (at 82.55 19.05 0)
-      (effects (font (size 1.27 1.27)) hide)
-    )
-    (pin "1")
-    (instances
-      (project "frankenstein_enlarger_controller"
-        (path "/1ba54f55-ab1c-4f2f-aaa2-6abd42790785/a070d1c7-4928-4ffb-b06d-351ae78e3b54"
-          (reference "#PWR057") (unit 1)
-        )
-      )
-    )
-  )
   (symbol (lib_id "power:GND") (at 104.775 45.72 270) (unit 1)
     (in_bom yes) (on_board yes) (dnp no) (fields_autoplaced)
@@
     )
   )
-  (symbol (lib_id "Jumper:Jumper_2_Open") (at 82.55 31.75 90) (unit 1)
-    (in_bom yes) (on_board yes) (dnp no) (fields_autoplaced)
-    (property "Reference" "JP2" (at 83.82 31.115 90)
-      (effects (font (size 1.27 1.27)) (justify right))
-    )
-    (property "Value" "DMX+Termination" (at 83.82 33.655 90)
-      (effects (font (size 1.27 1.27)) (justify right))
-    )
-    (property "Footprint" "Jumper:SolderJumper-2_P1.3mm_Open_RoundedPad1.0x1.5mm" (at 82.55 31.75 0)
-      (effects (font (size 1.27 1.27)) hide)
-    )
-    (property "Datasheet" "~" (at 82.55 31.75 0)
-      (effects (font (size 1.27 1.27)) hide)
-    )
-    (pin "1")
-    (pin "2")
-    (instances
-      (project "frankenstein_enlarger_controller"
-        (path "/1ba54f55-ab1c-4f2f-aaa2-6abd42790785/a070d1c7-4928-4ffb-b06d-351ae78e3b54"
-          (reference "JP2") (unit 1)
-        )
-      )
-    )
-  )
   (symbol (lib_id "power:GND") (at 67.945 58.42 90) (unit 1)
     (in_bom yes) (on_board yes) (dnp no)
@@
         (path "/1ba54f55-ab1c-4f2f-aaa2-6abd42790785/a070d1c7-4928-4ffb-b06d-351ae78e3b54"
           (reference "#PWR053") (unit 1)
-        )
-      )
-    )
-  )
-  (symbol (lib_id "Device:R") (at 82.55 22.86 0) (unit 1)
-    (in_bom yes) (on_board yes) (dnp no) (fields_autoplaced)
-    (property "Reference" "R114" (at 84.455 22.225 0)
-      (effects (font (size 1.27 1.27)) (justify left))
-    )
-    (property "Value" "120" (at 84.455 24.765 0)
-      (effects (font (size 1.27 1.27)) (justify left))
-    )
-    (property "Footprint" "Resistor_SMD:R_0402_1005Metric" (at 80.772 22.86 90)
-      (effects (font (size 1.27 1.27)) hide)
-    )
-    (property "Datasheet" "~" (at 82.55 22.86 0)
-      (effects (font (size 1.27 1.27)) hide)
-    )
-    (property "LCSC" "C25079" (at 82.55 22.86 0)
-      (effects (font (size 1.27 1.27)) hide)
-    )
-    (pin "1")
-    (pin "2")
-    (instances
-      (project "frankenstein_enlarger_controller"
-        (path "/1ba54f55-ab1c-4f2f-aaa2-6abd42790785/a070d1c7-4928-4ffb-b06d-351ae78e3b54"
-          (reference "R114") (unit 1)
         )
       )
@@
         )
       )
-    )
-  )
-  (symbol (lib_id "power:GND") (at 82.55 65.405 0) (unit 1)
-    (in_bom yes) (on_board yes) (dnp no) (fields_autoplaced)
-    (property "Reference" "#PWR058" (at 82.55 71.755 0)
-      (effects (font (size 1.27 1.27)) hide)
-    )
-    (property "Value" "GND" (at 82.55 70.485 0)
-      (effects (font (size 1.27 1.27)))
-    )
-    (property "Footprint" "" (at 82.55 65.405 0)
-      (effects (font (size 1.27 1.27)) hide)
-    )
-    (property "Datasheet" "" (at 82.55 65.405 0)
-      (effects (font (size 1.27 1.27)) hide)
-    )
-    (pin "1")
-    (instances
-      (project "frankenstein_enlarger_controller"
-        (path "/1ba54f55-ab1c-4f2f-aaa2-6abd42790785/a070d1c7-4928-4ffb-b06d-351ae78e3b54"
-          (reference "#PWR058") (unit 1)
-        )
-      )
