File: Input Devices.kicad_sch (KiCad schematic)
At the start: 26 parts, among them SW1 RotaryEncoder_Switch, SW2 RotaryEncoder_Switch, SW3 RotaryEncoder_Switch, SW5 E-SWITCH 5501M, SW6 E-SWITCH 5501M, SW7 E-SWITCH 5501M, SW8 E-SWITCH 5501M, U2 74HC595

Commit message: Implemented fixes/changes after @manawyrm review
Connections:
- net SW5: now also SW5.3 (C); no longer SW5.2 (C)
- net SW6: now also SW6.3 (C); no longer SW6.2 (C)
- net SW7: now also SW7.3 (C); no longer SW7.2 (C)
- net SW8: now also SW8.3 (C); no longer SW8.2 (C)
- no-connect marks 8 -> 9
Changed lines of the file:
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@@
   (junction (at 124.46 129.54) (diameter 0) (color 0 0 0 0)
   )
-  (no_connect (at 62.23 119.38))
-  (no_connect (at 62.23 167.64))
-  (no_connect (at 62.23 95.25))
+  (no_connect (at 62.23 115.57))
+  (no_connect (at 62.23 163.83))
+  (no_connect (at 52.705 107.95))
   (no_connect (at 114.3 106.68))
+  (no_connect (at 62.23 91.44))
   (no_connect (at 114.3 111.76))
+  (no_connect (at 62.23 139.7))
   (no_connect (at 114.3 114.3))
   (no_connect (at 114.3 109.22))
-  (no_connect (at 62.23 143.51))
   (wire (pts (xy 114.3 119.38) (xy 101.6 119.38))
     (stroke (width 0) (type default))
@@
     (effects (font (size 1.27 1.27)) (justify right))
   )
-  (hierarchical_label "SW6" (shape input) (at 62.23 115.57 0) (fields_autoplaced)
+  (hierarchical_label "SW6" (shape input) (at 62.23 119.38 0) (fields_autoplaced)
     (effects (font (size 1.27 1.27)) (justify left))
   )
@@
     (effects (font (size 1.27 1.27)) (justify right))
   )
-  (hierarchical_label "SW5" (shape input) (at 62.23 91.44 0) (fields_autoplaced)
+  (hierarchical_label "SW5" (shape input) (at 62.23 95.25 0) (fields_autoplaced)
     (effects (font (size 1.27 1.27)) (justify left))
   )
@@
     (effects (font (size 1.27 1.27)) (justify left))
   )
-  (hierarchical_label "SW8" (shape input) (at 62.23 163.83 0) (fields_autoplaced)
+  (hierarchical_label "SW8" (shape input) (at 62.23 167.64 0) (fields_autoplaced)
     (effects (font (size 1.27 1.27)) (justify left))
   )
@@
     (effects (font (size 1.27 1.27)) (justify right))
   )
-  (hierarchical_label "SW7" (shape input) (at 62.23 139.7 0) (fields_autoplaced)
-    (effects (font (size 1.27 1.27)) (justify left))
-  )
+  (hierarchical_label "SW7" (shape input) (at 62.23 143.51 0) (fields_autoplaced)
+    (effects (font (size 1.27 1.27)) (justify left))
+  )

Commit message: Consolidated Hardware on single board
Parts:
- C59: renamed from C1; value 100n -> C
- R138: renamed from R4; value 120 -> R
- R139: renamed from R3; value 120 -> R
- R140: renamed from R2; value 120 -> R
- R141: renamed from R1; value 120 -> R
- R73, R74, R75, R76, R77, R78, R79, R80, R81: value 5.1k -> R
- renumbered SW6 to SW10, SW7 to SW11, SW8 to SW12, SW5 to SW9, U2 to U33
Other:
- company: (none) -> wirkbetrieb.net / Tom Eichhorn
- title: (none) -> Frankenstein Controller
