File: USB-C_PD.kicad_sch (KiCad schematic)
At the start: 16 parts, among them Q1 DMP3013SFV-7, Q2 DMP3013SFV-7, U7 CYPD3177-24LQXQ

Commit message: Tie VBUS_FET_EN and SAFE_PWR_EN together
Parts:
- R25: value 10k 0603 -> 1k 0603
Connections:
- net at R30.2, U7.3 (VBUS_FET_EN): now also U7.4 (SAFE_PWR_EN)
- no-connect marks 7 -> 6
Changed lines of the file:
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@@
   (junction (at 161.29 125.73) (diameter 0) (color 0 0 0 0)
+  )
+  (junction (at 101.6 73.66) (diameter 0) (color 0 0 0 0)
   )
   (junction (at 142.24 143.51) (diameter 0) (color 0 0 0 0)
@@
   (no_connect (at 104.14 96.52))
   (no_connect (at 104.14 91.44))
-  (no_connect (at 104.14 76.2))
   (wire (pts (xy 116.84 48.26) (xy 121.92 48.26))
     (stroke (width 0) (type default))
@@
     (stroke (width 0) (type default))
   )
+  (wire (pts (xy 104.14 76.2) (xy 101.6 76.2))
+    (stroke (width 0) (type default))
+  )
   (wire (pts (xy 116.84 39.37) (xy 116.84 48.26))
     (stroke (width 0) (type default))
@@
     (stroke (width 0) (type default))
   )
-  (wire (pts (xy 92.71 73.66) (xy 104.14 73.66))
+  (wire (pts (xy 92.71 73.66) (xy 101.6 73.66))
+    (stroke (width 0) (type default))
+  )
+  (wire (pts (xy 101.6 73.66) (xy 104.14 73.66))
     (stroke (width 0) (type default))
   )
@@
   )
   (wire (pts (xy 104.14 119.38) (xy 104.14 165.735))
+    (stroke (width 0) (type default))
+  )
+  (wire (pts (xy 101.6 76.2) (xy 101.6 73.66))
     (stroke (width 0) (type default))
   )
@@
       (effects (font (size 1.27 1.27)))
     )
-    (property "Value" "10k 0603" (at 111.76 27.94 0)
-      (effects (font (size 1.27 1.27)))
-    )
+    (property "Value" "1k 0603" (at 111.76 27.94 0)
+      (effects (font (size 1.27 1.27)))
+    )
