File: picoassembly.kicad_sch (KiCad schematic)
At the start: 24 parts, among them SW10 TS-1187A-B-A-B, SW9 TS-1187A-B-A-B, U17 W25Q128JVS, U18 RP2040, Y2 Crystal_GND24

Commit message: Tie VBUS_FET_EN and SAFE_PWR_EN together
Parts:
- renumbered C29 to C1, C27 to C10, C35 to C11, C28 to C12, C30 to C13, C36 to C14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
